File: TFG.kicad_sch (KiCad schematic)
At the start: 37 parts, among them J1 Voltaje Input, J2 IDC-header, U2 LM2596, U3 ESP-WROOM-32, U4 LM339N, U5 LM339N, U6 ESP-WROOM-32

Commit message: update sq
Parts:
- removed U3: ESP-WROOM-32, NMDA-lib:MODULE_ESP32_DEVKIT_V1, symbol NMDA-lib:esp32_38_pins
- added U1: ESP32-DEVKIT-V1, NMDA-lib:MODULE_ESP32_DEVKIT_V1, symbol ESP32-DEVKIT-V1:ESP32-DEVKIT-V1
- D1, D2, D3: value 1N4007 -> 2N3896
- R13, R14, R15: value 22k -> 33k
Connections:
- net 3.3V: now also U1.1 (3V3)
- net GND: now also U1.2 (GND), U1.29 (GND)
- net I2C_SCL: now also U1.14 (D22)
- net I2C_SDA: now also U1.11 (D21)
- net PULSE_IN_CH01: now also U1.8 (D5)
- net PULSE_IN_CH02: now also U1.26 (D14)
- net PULSE_IN_CH03: now also U1.3 (D15)
- net TUBE1: now also J2.3 (Pin_3); no longer J2.7 (Pin_7)
- net TUBE3: now also J2.7 (Pin_7); no longer J2.3 (Pin_3)
- no-connect marks 33 -> 27
